File: pcb/macropad.kicad_sch (KiCad schematic)
At the start: 40 parts, among them SW1 RotaryEncoder, SW10 SW_Push, SW2 SW_Push, SW3 SW_Push, SW4 SW_Push, SW5 SW_Push, SW6 SW_Push, SW7 SW_Push, SW8 SW_Push, SW9 SW_Push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

Commit message: switched to the correct diode footprint
Parts:
- D17, D18, D19, D20, D21, D22, D23, D24, D25, D26, D27, D28: footprint Diode_THT:D_T-1_P5.08mm_Horizontal -> Diode_THT:D_DO-35_SOD27_P7.62mm_Horizontal
Changed lines of the file:
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@@
 			)
 		)
-		(property "Footprint" "Diode_THT:D_T-1_P5.08mm_Horizontal"
+		(property "Footprint" "Diode_THT:D_DO-35_SOD27_P7.62mm_Horizontal"
 			(at 58.42 60.96 90)
 			(effects
@@
 			)
 		)
-		(property "Footprint" "Diode_THT:D_T-1_P5.08mm_Horizontal"
+		(property "Footprint" "Diode_THT:D_DO-35_SOD27_P7.62mm_Horizontal"
 			(at 58.42 44.45 90)
 			(effects
@@
 			)
 		)
-		(property "Footprint" "Diode_THT:D_T-1_P5.08mm_Horizontal"
+		(property "Footprint" "Diode_THT:D_DO-35_SOD27_P7.62mm_Horizontal"
 			(at 72.39 60.96 90)
 			(effects
@@
 			)
 		)
-		(property "Footprint" "Diode_THT:D_T-1_P5.08mm_Horizontal"
+		(property "Footprint" "Diode_THT:D_DO-35_SOD27_P7.62mm_Horizontal"
 			(at 57.15 99.06 90)
 			(effects
@@
 			)
 		)
-		(property "Footprint" "Diode_THT:D_T-1_P5.08mm_Horizontal"
+		(property "Footprint" "Diode_THT:D_DO-35_SOD27_P7.62mm_Horizontal"
 			(at 58.42 29.21 90)
 			(effects
@@
 			)
 		)
-		(property "Footprint" "Diode_THT:D_T-1_P5.08mm_Horizontal"
+		(property "Footprint" "Diode_THT:D_DO-35_SOD27_P7.62mm_Horizontal"
 			(at 52.07 99.06 90)
 			(effects
@@
 			)
 		)
-		(property "Footprint" "Diode_THT:D_T-1_P5.08mm_Horizontal"
+		(property "Footprint" "Diode_THT:D_DO-35_SOD27_P7.62mm_Horizontal"
 			(at 44.45 44.45 90)
 			(effects
@@
 			)
 		)
-		(property "Footprint" "Diode_THT:D_T-1_P5.08mm_Horizontal"
+		(property "Footprint" "Diode_THT:D_DO-35_SOD27_P7.62mm_Horizontal"
 			(at 44.45 29.21 90)
 			(effects
@@
 			)
 		)
-		(property "Footprint" "Diode_THT:D_T-1_P5.08mm_Horizontal"
+		(property "Footprint" "Diode_THT:D_DO-35_SOD27_P7.62mm_Horizontal"
 			(at 72.39 44.45 90)
 			(effects
@@
 			)
 		)
-		(property "Footprint" "Diode_THT:D_T-1_P5.08mm_Horizontal"
+		(property "Footprint" "Diode_THT:D_DO-35_SOD27_P7.62mm_Horizontal"
 			(at 71.12 99.06 90)
 			(effects
@@
 			)
 		)
-		(property "Footprint" "Diode_THT:D_T-1_P5.08mm_Horizontal"
+		(property "Footprint" "Diode_THT:D_DO-35_SOD27_P7.62mm_Horizontal"
 			(at 72.39 29.21 90)
 			(effects
@@
 			)
 		)
-		(property "Footprint" "Diode_THT:D_T-1_P5.08mm_Horizontal"
+		(property "Footprint" "Diode_THT:D_DO-35_SOD27_P7.62mm_Horizontal"
 			(at 44.45 60.96 90)
 			(effects
